File: Isolated IO.kicad_sch (KiCad schematic)
At the start: 2 parts, among them U3 LTC2861

Commit message: Finished capturing schematics
Parts:
- removed C3: C, symbol Device:C
- removed U3: LTC2861, Package_SO:SSOP-28_5.3x10.2mm_P0.65mm, symbol Interface_UART:LTC2861
- added C1, C2: C, symbol Device:C
- added U2: Si8641BB-B-IU, Package_SO:QSOP-16_3.9x4.9mm_P0.635mm, symbol Isolator:Si8641BB-B-IU
Connections:
- net GND DUT: now also C2.2, U2.15 (GND2), U2.9 (GND2)
- new net GND USB: C1.2, U2.2 (GND1), U2.8 (GND1)
- new net In1 A: U2.3 (A1)
- new net In2 A: U2.4 (A2)
- new net In3 A: U2.5 (A3)
- new net In4 B: U2.11 (B4)
- new net Out1 B: U2.14 (B1)
- new net Out2 B: U2.13 (B2)
- new net Out3 B: U2.12 (B3)
- new net Out4 A: U2.6 (A4)
- new net Power A: C1.1, U2.1 (VDD1), U2.7 (EN1)
- new net Power B: C2.1, U2.10 (EN2), U2.16 (VDD2)

Commit message: Power & Level Translation
Isolated 5VDC changed and a 3.3VDC LDO was added. The original 5VDC was too expensive and big. The new one is still both, but less so.
The level translator is now a dedicated IC instead of MOSFETs. I was having trouble making it work the way I wanted.
Changed lines of the file:
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@@
 	)
 	(hierarchical_label "Power B"
-		(shape input)
+		(shape output)
 		(at 152.4 63.5 0)
 		(fields_autoplaced yes)
@@
 		(dnp no)
 		(fields_autoplaced yes)
-		(property "Reference" "#PWR010"
+		(property "Reference" "#PWR014"
 			(at 111.76 113.03 0)
 			(effects
@@
 			(project "Isolated Com Port"
 				(path "/736fe05f-3e80-4c58-a4b9-c0a7b5ae4e97/2bf4cea1-1398-4e51-b092-f0619f1c193c"
-					(reference "#PWR010")
+					(reference "#PWR014")
 					(unit 1)
 				)
@@
 		(dnp no)
 		(fields_autoplaced yes)
-		(property "Reference" "#PWR012"
+		(property "Reference" "#PWR016"
 			(at 147.32 82.55 0)
 			(effects
@@
 			(project "Isolated Com Port"
 				(path "/736fe05f-3e80-4c58-a4b9-c0a7b5ae4e97/2bf4cea1-1398-4e51-b092-f0619f1c193c"
-					(reference "#PWR012")
+					(reference "#PWR016")
 					(unit 1)
 				)
@@
 		(dnp no)
 		(fields_autoplaced yes)
-		(property "Reference" "#PWR011"
+		(property "Reference" "#PWR013"
 			(at 101.6 82.55 0)
 			(effects
@@
 			(project "Isolated Com Port"
 				(path "/736fe05f-3e80-4c58-a4b9-c0a7b5ae4e97/2bf4cea1-1398-4e51-b092-f0619f1c193c"
-					(reference "#PWR011")
+					(reference "#PWR013")
 					(unit 1)
 				)
@@
 		(dnp no)
 		(fields_autoplaced yes)
-		(property "Reference" "#PWR09"
+		(property "Reference" "#PWR015"
 			(at 137.16 113.03 0)
 			(effects
@@
 			(project "Isolated Com Port"
 				(path "/736fe05f-3e80-4c58-a4b9-c0a7b5ae4e97/2bf4cea1-1398-4e51-b092-f0619f1c193c"
-					(reference "#PWR09")
+					(reference "#PWR015")
 					(unit 1)
 				)
@@
 		(on_board yes)
 		(dnp no)
-		(fields_autoplaced yes)
 		(property "Reference" "U2"
-			(at 124.46 73.66 0)
+			(at 118.11 77.47 0)
 			(effects
 				(font
@@
 		)
 		(property "Value" "Si8641BB-B-IU"
-			(at 124.46 76.2 0)
-			(effects
-				(font
+			(at 124.46 105.41 0)
+			(effects
+				(font
