File: RS485.kicad_sch (KiCad schematic)
At the start: 2 parts, among them U3 LTC2861

Commit message: Power & Level Translation
Isolated 5VDC changed and a 3.3VDC LDO was added. The original 5VDC was too expensive and big. The new one is still both, but less so.
The level translator is now a dedicated IC instead of MOSFETs. I was having trouble making it work the way I wanted.
Parts:
- renumbered C3 to C7, U3 to U5
Changed lines of the file:
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@@
 	)
 	(hierarchical_label "Termination"
-		(shape output)
+		(shape input)
 		(at 149.86 114.3 0)
 		(fields_autoplaced yes)
@@
 	)
 	(hierarchical_label "TX Enable"
-		(shape output)
+		(shape input)
 		(at 96.52 119.38 180)
 		(fields_autoplaced yes)
@@
 		(dnp no)
 		(fields_autoplaced yes)
-		(property "Reference" "#PWR017"
+		(property "Reference" "#PWR031"
 			(at 119.38 105.41 0)
 			(effects
@@
 			(project "Isolated Com Port"
 				(path "/736fe05f-3e80-4c58-a4b9-c0a7b5ae4e97/70b8d09c-0e85-4c64-81a9-47ae182320c8"
-					(reference "#PWR017")
+					(reference "#PWR031")
 					(unit 1)
 				)
@@
 		(on_board yes)
 		(dnp no)
-		(property "Reference" "U3"
+		(property "Reference" "U5"
 			(at 129.8859 105.41 0)
 			(effects
@@
 			(project "Isolated Com Port"
 				(path "/736fe05f-3e80-4c58-a4b9-c0a7b5ae4e97/70b8d09c-0e85-4c64-81a9-47ae182320c8"
-					(reference "U3")
+					(reference "U5")
 					(unit 1)
 				)
@@
 		(dnp no)
 		(fields_autoplaced yes)
-		(property "Reference" "#PWR025"
+		(property "Reference" "#PWR029"
 			(at 66.04 128.27 0)
 			(effects
@@
 			(project "Isolated Com Port"
 				(path "/736fe05f-3e80-4c58-a4b9-c0a7b5ae4e97/70b8d09c-0e85-4c64-81a9-47ae182320c8"
-					(reference "#PWR025")
+					(reference "#PWR029")
 					(unit 1)
 				)
@@
 		(dnp no)
 		(fields_autoplaced yes)
-		(property "Reference" "C3"
+		(property "Reference" "C7"
 			(at 69.85 114.2999 0)
 			(effects
@@
 			(project "Isolated Com Port"
 				(path "/736fe05f-3e80-4c58-a4b9-c0a7b5ae4e97/70b8d09c-0e85-4c64-81a9-47ae182320c8"
-					(reference "C3")
+					(reference "C7")
 					(unit 1)
 				)
@@
 		(dnp no)
 		(fields_autoplaced yes)
-		(property "Reference" "#PWR024"
+		(property "Reference" "#PWR030"
 			(at 104.14 143.51 0)
 			(effects
@@
 			(project "Isolated Com Port"
 				(path "/736fe05f-3e80-4c58-a4b9-c0a7b5ae4e97/70b8d09c-0e85-4c64-81a9-47ae182320c8"
-					(reference "#PWR024")
+					(reference "#PWR030")
 					(unit 1)
 				)
@@
 		(dnp no)
 		(fields_autoplaced yes)
-		(property "Reference" "#PWR018"
+		(property "Reference" "#PWR032"
 			(at 119.38 148.59 0)
 			(effects
@@
 			(project "Isolated Com Port"
 				(path "/736fe05f-3e80-4c58-a4b9-c0a7b5ae4e97/70b8d09c-0e85-4c64-81a9-47ae182320c8"
-					(reference "#PWR018")
+					(reference "#PWR032")
 					(unit 1)
 				)
@@
 		(dnp no)
 		(fields_autoplaced yes)
-		(property "Reference" "#PWR027"
+		(property "Reference" "#PWR028"
 			(at 66.04 113.03 0)
 			(effects
@@
 			(project "Isolated Com Port"
 				(path "/736fe05f-3e80-4c58-a4b9-c0a7b5ae4e97/70b8d09c-0e85-4c64-81a9-47ae182320c8"
-					(reference "#PWR027")
-					(unit 1)
-				)
+					(reference "#PWR028")
+					(unit 1)
+				)
